Commit message: 20231030

File: pick_robot_description/urdf/epick/urdf/epick_single_suction_cup.xacro (robot description, xacro)
@@ -3,4 +3,5 @@
   <!-- Include EPick Body and helper macros -->
   <xacro:include filename="epick_body.xacro"/>
+  <!-- removed by gerard -->
 <!--
   <xacro:include filename="$(find epick_description)/urdf/epick_driver_ros2_control.xacro" />
@@ -79,5 +80,5 @@
     <!-- To allow MoveIt to actuate the gripper as part of a trajectory, we need to include a fake "joint" in the URDF corresponding to the Epick's vacuum state. -->
     <link name="${prefix}epick_vacuum_state"/>
-    <joint name="gripper" type="revolute">
+    <joint name="gripper" type="fixed"> <!-- changed by gerard -->
       <origin xyz="0 0 0" rpy="0 0 0"/>
       <parent link="${prefix}epick_tcp"/>
