Commit message: 20240409

File: pick_robot_description/urdf/pick_robot.urdf.xacro (robot description, xacro)
@@ -14,9 +14,39 @@
    <xacro:arg name="physical_params" default="$(find pick_robot_description)/config/$(arg ur_type)/physical_parameters.yaml"/>
    <xacro:arg name="visual_params" default="$(find pick_robot_description)/config/$(arg ur_type)/visual_parameters.yaml"/>
+   <xacro:arg name="transmission_hw_interface" default=""/>
    <xacro:arg name="safety_limits" default="false"/>
    <xacro:arg name="safety_pos_margin" default="0.15"/>
    <xacro:arg name="safety_k_position" default="20"/>
-   <!--When using gazebo simulations absolute paths are necessary.-->
-   <xacro:arg name="force_abs_paths" default="false" />
+   <!-- ros2_control related parameters -->
+   <xacro:arg name="headless_mode" default="false" />
+   <xacro:arg name="robot_ip" default="0.0.0.0" />
+   <xacro:arg name="script_filename" default=""/>
+   <xacro:arg name="output_recipe_filename" default=""/>
+   <xacro:arg name="input_recipe_filename" default=""/>
+   <xacro:arg name="reverse_ip" default="0.0.0.0"/>
+   <xacro:arg name="script_command_port" default="50004"/>
+   <xacro:arg name="reverse_port" default="50001"/>
+   <xacro:arg name="script_sender_port" default="50002"/>
+   <xacro:arg name="trajectory_port" default="50003"/>
+   <!--   tool communication related parameters-->
+   <xacro:arg name="use_tool_communication" default="false" />
+   <xacro:arg name="tool_voltage" default="0" />
+   <xacro:arg name="tool_parity" default="0" />
+   <xacro:arg name="tool_baud_rate" default="115200" />
+   <xacro:arg name="tool_stop_bits" default="1" />
+   <xacro:arg name="tool_rx_idle_chars" default="1.5" />
+   <xacro:arg name="tool_tx_idle_chars" default="3.5" />
+   <xacro:arg name="tool_device_name" default="/tmp/ttyUR" />
+   <xacro:arg name="tool_tcp_port" default="54321" />
+     <!-- Simulation parameters -->
+   <xacro:arg name="use_fake_hardware" default="false" />
+   <xacro:arg name="fake_sensor_commands" default="false" />
+   <xacro:arg name="sim_gazebo" default="false" />
+   <xacro:arg name="sim_ignition" default="false" />
+   <xacro:arg name="simulation_controllers" default="" />
+   <!-- initial position for simulations (Fake Hardware, Gazebo, Ignition) -->
+   <xacro:arg name="initial_positions_file" default="$(find ur_description)/config/initial_positions.yaml"/>
+   <!-- convert to property to use substitution in function -->
+   <xacro:property name="initial_positions_file" default="$(arg initial_positions_file)"/>
    <!-- create link fixed to the "world" -->
    <link name="world" />
@@ -30,7 +60,32 @@
      physical_parameters_file="$(arg physical_params)"
      visual_parameters_file="$(arg visual_params)"
+     transmission_hw_interface="$(arg transmission_hw_interface)"
      safety_limits="$(arg safety_limits)"
      safety_pos_margin="$(arg safety_pos_margin)"
      safety_k_position="$(arg safety_k_position)"
+     use_fake_hardware="$(arg use_fake_hardware)"
+     fake_sensor_commands="$(arg fake_sensor_commands)"
+     sim_gazebo="$(arg sim_gazebo)"
+     sim_ignition="$(arg sim_ignition)"
+     headless_mode="$(arg headless_mode)"
+     initial_positions="${xacro.load_yaml(initial_positions_file)}"
+     use_tool_communication="$(arg use_tool_communication)"
+     tool_voltage="$(arg tool_voltage)"
+     tool_parity="$(arg tool_parity)"
+     tool_baud_rate="$(arg tool_baud_rate)"
+     tool_stop_bits="$(arg tool_stop_bits)"
+     tool_rx_idle_chars="$(arg tool_rx_idle_chars)"
+     tool_tx_idle_chars="$(arg tool_tx_idle_chars)"
+     tool_device_name="$(arg tool_device_name)"
+     tool_tcp_port="$(arg tool_tcp_port)"
+     robot_ip="$(arg robot_ip)"
+     script_filename="$(arg script_filename)"
+     output_recipe_filename="$(arg output_recipe_filename)"
+     input_recipe_filename="$(arg input_recipe_filename)"
+     reverse_ip="$(arg reverse_ip)"
+     script_command_port="$(arg script_command_port)"
+     reverse_port="$(arg reverse_port)"
+     script_sender_port="$(arg script_sender_port)"
+     trajectory_port="$(arg trajectory_port)"
      >
      <origin xyz="0 0 0" rpy="0 0 0" />          <!-- position robot in the world -->
@@ -123,5 +178,5 @@
     <origin xyz="0.0 0.00 0.0" rpy="0 0 0"/>
   </joint>
-      <xacro:arg name="camera_name"   default="oak" />
+    <xacro:arg name="camera_name"   default="oak" />
     <xacro:arg name="camera_model"  default="OAK-D" />
     <xacro:arg name="base_frame"    default="oak-d_frame" />
@@ -137,9 +192,6 @@
     <xacro:arg name="b"             default="0.0" />
     <xacro:arg name="a"             default="1.0" />
-    <!--
     <xacro:include filename="$(find depthai_descriptions)/urdf/include/depthai_macro.urdf.xacro"/>
-    -->
-    <xacro:include filename="$(find depthai_descriptions)/urdf/include/base_macro.urdf.xacro"/>
-    <xacro:base camera_name = "$(arg camera_name)"
+    <xacro:depthai_camera camera_name = "$(arg camera_name)"
                           parent = "$(arg parent_frame)"
                           camera_model = "$(arg camera_model)"
@@ -151,5 +203,4 @@
                           cam_pitch = "$(arg cam_pitch)"
                           cam_yaw = "$(arg cam_yaw)"
-                          has_imu = "false"
                           r = "$(arg r)"
                           g = "$(arg g)"
@@ -164,3 +215,24 @@
   <xacro:epick_single_suction_cup parent="beugel_tool" use_fake_hardware="true"/>
 -->
+   <xacro:if value="$(arg sim_gazebo)">
+    <!-- Gazebo plugins -->
+    <gazebo reference="world">
+    </gazebo>
+    <gazebo>
+      <plugin filename="libgazebo_ros2_control.so" name="gazebo_ros2_control">
+        <parameters>$(arg simulation_controllers)</parameters>
+      </plugin>
+    </gazebo>
+  </xacro:if>
+  <xacro:if value="$(arg sim_ignition)">
+    <!-- Gazebo plugins -->
+    <gazebo reference="world">
+    </gazebo>
+    <gazebo>
+      <plugin filename="libign_ros2_control-system.so" name="ign_ros2_control::IgnitionROS2ControlPlugin">
+        <parameters>$(arg simulation_controllers)</parameters>
+        <controller_manager_node_name>$(arg tf_prefix)controller_manager</controller_manager_node_name>
+      </plugin>
+    </gazebo>
+  </xacro:if>
 </robot>

Commit message: 20240414

File: pick_robot_description/urdf/pick_robot.urdf.xacro (robot description, xacro)
@@ -127,10 +127,10 @@
       <xacro:box_inertia m="10" x="1.1" y="0.7" z="0.03"/>
     </inertial>
-    <collision>
+        <collision>
       <geometry>
         <box size="0.7 1.1 0.03" />
       </geometry>
     </collision>
-  </link>
+      </link>
   <joint name="baseplate_joint" type="fixed">
     <origin xyz="0 0 0" />
@@ -150,10 +150,10 @@
       <xacro:box_inertia m="1" x="0.3" y="0.3" z="0.012"/>
     </inertial>
-    <collision>
+        <collision>
       <geometry>
         <box size="0.3 0.3 0.012" />
       </geometry>
     </collision>
-  </link>
+      </link>
   <joint name="mountingplate_joint" type="fixed">
     <origin xyz="-0.2 0.0 0.021" />
