Commit message: 20231108-1

File: pick_robot_description/urdf/beugel/urdf/BeugelArrow.urdf.xacro (robot description, xacro)
@@ -4,5 +4,5 @@
      For more information, please see http://wiki.ros.org/sw_urdf_exporter -->
 <robot xmlns:xacro="http://wiki.ros.org/xacro">
-  <xacro:macro name="beugel">
+  <xacro:macro name="beugel_arrow">
   <link name="beugel_link"/>
  <joint name="beugel_link_to_beugel_link_mesh" type="fixed">
@@ -70,4 +70,10 @@
         <origin xyz="0.00 0 0.033" rpy="0 ${-pi/2} ${pi/2}"/>
     </joint>
-  </xacro:macro>
+    <link name="arrow_tcp"/>
+    <joint name="beugel_link_mesh_to_arrow_tcp" type="fixed">
+        <parent link="beugel_link_mesh" />
+        <child link="arrow_tcp" />
+        <origin xyz="0.0 0.00 0.04308" rpy="0 0 0"/>
+      </joint>
+    </xacro:macro>
 </robot>

File: pick_robot_description/urdf/pick_robot.urdf.xacro (robot description, xacro)
@@ -7,5 +7,5 @@
    <!-- possible 'ur_type' values: ur3, ur3e, ur5, ur5e, ur10, ur10e, ur16e, ur20 -->
    <!-- the default value should raise an error in case this was called without defining the type -->
-   <xacro:arg name="ur_type" default="ur5e"/>
+   <xacro:arg name="ur_type" default="ur3"/>
    <!-- parameters -->
    <xacro:arg name="tf_prefix" default="" />
@@ -175,5 +175,5 @@
   <!-- bracket/beugel -->
   <xacro:include filename="beugel/urdf/BeugelArrow.urdf.xacro" />
-  <xacro:beugel/>
+  <xacro:beugel_arrow/>
   <!-- tool0 to beugel_base_position -->
   <!-- cahnge these valuse to place the beugel on the right position -->

Commit message: 20231109

File: pick_robot_description/urdf/beugel/urdf/BeugelArrow.urdf.xacro (robot description, xacro)
@@ -32,5 +32,7 @@
       <geometry>
         <mesh
-          filename="package://pick_robot_description/urdf/beugel/meshes/Beugel-OAK-D-Arrow.SLDPRT.STL" />
+          filename="package://pick_robot_description/urdf/beugel/meshes/Beugel-OAK-D-Arrow.SLDPRT.STL"
+          scale="0.0005 0.0005 0.0005"
+           />
       </geometry>
       <material name="BeugelColor">
@@ -74,5 +76,5 @@
         <parent link="beugel_link_mesh" />
         <child link="arrow_tcp" />
-        <origin xyz="0.0 0.00 0.04308" rpy="0 0 0"/>
+        <origin xyz=" 0.0 0.04308 0.00 " rpy="0 0 0"/>
       </joint>
     </xacro:macro>

Commit message: 20231111

File: pick_robot_description/urdf/beugel/urdf/BeugelArrow.urdf.xacro (robot description, xacro)
@@ -33,9 +33,9 @@
         <mesh
           filename="package://pick_robot_description/urdf/beugel/meshes/Beugel-OAK-D-Arrow.SLDPRT.STL"
-          scale="0.0005 0.0005 0.0005"
+          scale="0.001 0.001 0.001"
            />
       </geometry>
       <material name="BeugelColor">
-        <color rgba="0.25 0.25 0.25 1" />
+        <color rgba="0 0 1 1" />
         <!--
         <texture

File: pick_robot_description/urdf/pick_robot.urdf.xacro (robot description, xacro)
@@ -173,7 +173,17 @@
     <origin xyz="0.0 0.0 0.01" rpy="0.0 0.0 ${pi}"/>
   </joint>
+  <link name= "pick_tcp" />
   <!-- bracket/beugel -->
   <xacro:include filename="beugel/urdf/BeugelArrow.urdf.xacro" />
   <xacro:beugel_arrow/>
+  <joint name="pick_tcp_to_pick_tcp" type="fixed">
+    <parent link="arrow_tcp" />
+    <child link="pick_tcp" />
+    <origin xyz="0.0 0.0 0.0" rpy="0.0 0.0 0.0"/>
+  </joint>
+  <!--
+  <xacro:include filename="beugel/urdf/Beugel.urdf.xacro" />
+  <xacro:beugel/>
+  -->
   <!-- tool0 to beugel_base_position -->
   <!-- cahnge these valuse to place the beugel on the right position -->

Commit message: 20240304

File: pick_robot_description/urdf/beugel/urdf/BeugelArrow.urdf.xacro (robot description, xacro)
@@ -9,5 +9,8 @@
     <parent link="beugel_link" />
     <child link="beugel_link_mesh" />
+    <!--
     <origin xyz="0.0 0.00 0.01" rpy="${pi/2} 0 ${pi}"/>
+    -->
+    <origin xyz="0.0 0.00 0.01" rpy="0 0 0"/>
   </joint>
   <link name="beugel_link_mesh">
@@ -27,10 +30,13 @@
     </inertial>
     <visual>
+        <!--
+        DE ORGIN GETALLEN BEGRIJP IK NIET
+        -->
       <origin
-        xyz="0 0 0"
-        rpy="${pi/2} 0 0" />
+       xyz="0.04 -0.04  0.04308"
+       rpy="0 ${pi} 0" />
       <geometry>
         <mesh
-          filename="package://pick_robot_description/urdf/beugel/meshes/Beugel-OAK-D-Arrow.SLDPRT.STL"
+          filename="package://pick_robot_description/urdf/beugel/meshes/Beugel-OAK-D-Arrow.STL"
           scale="0.001 0.001 0.001"
            />
@@ -45,10 +51,15 @@
     </visual>
     <collision>
+        <!--
+        DE ORGIN GETALLEN BEGRIJP IK NIET
+        -->
       <origin
-        xyz="0 0 0"
-        rpy="${pi/2} 0 0" />
+       xyz="0.04 -0.04  0.04308"
+        rpy="0 ${pi} 0" />
       <geometry>
         <mesh
-          filename="package://pick_robot_description/urdf/beugel/meshes/Beugel-OAK-D-Arrow.SLDPRT.STL" />
+          filename="package://pick_robot_description/urdf/beugel/meshes/Beugel-OAK-D-Arrow.STL"
+          scale="0.001 0.001 0.001"
+          />
       </geometry>
     </collision>
@@ -76,5 +87,5 @@
         <parent link="beugel_link_mesh" />
         <child link="arrow_tcp" />
-        <origin xyz=" 0.0 0.04308 0.00 " rpy="0 0 0"/>
+        <origin xyz=" 0.0  0.00 0.04308" rpy="0 0 0"/>
       </joint>
     </xacro:macro>
