Commit message: 20240516

File: pick_robot_description/urdf/beugel/urdf/Beugel.urdf.xacro (robot description, xacro)
@@ -5,7 +5,7 @@
 <robot xmlns:xacro="http://wiki.ros.org/xacro">
   <xacro:macro name="beugel">
-  <link name="beugel_link"/>
+  <link name="beugel_base_link"/>
  <joint name="beugel_link_to_beugel_link_mesh" type="fixed">
-    <parent link="beugel_link" />
+    <parent link="beugel_base_link" />
     <child link="beugel_link_mesh" />
     <origin xyz="0.0 0.00 0.01" rpy="${pi/2} 0 ${pi}"/>
@@ -56,5 +56,5 @@
   <link name="beugel_tool"/>
  <joint name="beugel_link_to_beugel_tool" type="fixed">
-    <parent link="beugel_link" />
+    <parent link="beugel_base_link" />
     <child link="beugel_tool" />
     <origin xyz="0.0 0.00 0.005" rpy="0 0 0"/>
@@ -62,5 +62,5 @@
     <link name="beugel_camera_pre"/>
     <joint name="beugel_link_to_beugel_camera_pre" type="fixed">
-        <parent link="beugel_link" />
+        <parent link="beugel_base_link" />
         <child link="beugel_camera_pre" />
         <origin xyz="0.00 0.04634 ${0.005-0.00254}" rpy="${-pi/6*1} 0 0"/>

File: pick_robot_description/urdf/beugel/urdf/BeugelWithArrow.urdf.xacro (robot description, xacro)
@@ -4,15 +4,18 @@
      For more information, please see http://wiki.ros.org/sw_urdf_exporter -->
 <robot xmlns:xacro="http://wiki.ros.org/xacro">
-  <xacro:macro name="beugel_arrow">
-  <link name="beugel_link"/>
- <joint name="beugel_link_to_beugel_link_mesh" type="fixed">
-    <parent link="beugel_link" />
-    <child link="beugel_link_mesh" />
+  <xacro:macro name="beugel_with_arrow">
+  <link name="beugel_base_link"/>
+ <joint name="arrow_link_to_arrow_link_mesh" type="fixed">
+    <parent link="beugel_base_link" />
+    <child link="arrow_link_mesh" />
     <!--
     <origin xyz="0.0 0.00 0.01" rpy="${pi/2} 0 ${pi}"/>
     -->
+    <!--
+    <origin xyz="0.00 0.04634 ${0.005-0.00254}" rpy="${-pi/6*1} 0 0"/>
+    -->
     <origin xyz="0.0 0.00 0.01" rpy="0 0 0"/>
   </joint>
-  <link name="beugel_link_mesh">
+  <link name="arrow_link_mesh">
     <inertial>
       <origin
@@ -67,5 +70,5 @@
   <link name="beugel_tool"/>
  <joint name="beugel_link_to_beugel_tool" type="fixed">
-    <parent link="beugel_link" />
+    <parent link="beugel_base_link" />
     <child link="beugel_tool" />
     <origin xyz="0.0 0.00 0.005" rpy="0 0 0"/>
@@ -73,5 +76,5 @@
     <link name="beugel_camera_pre"/>
     <joint name="beugel_link_to_beugel_camera_pre" type="fixed">
-        <parent link="beugel_link" />
+        <parent link="beugel_base_link" />
         <child link="beugel_camera_pre" />
         <origin xyz="0.00 0.04634 ${0.005-0.00254}" rpy="${-pi/6*1} 0 0"/>
@@ -84,6 +87,6 @@
     </joint>
     <link name="arrow_tcp"/>
-    <joint name="beugel_link_mesh_to_arrow_tcp" type="fixed">
-        <parent link="beugel_link_mesh" />
+    <joint name="arrow_link_mesh_to_arrow_tcp" type="fixed">
+        <parent link="arrow_link_mesh" />
         <child link="arrow_tcp" />
         <origin xyz=" 0.0  0.00 0.04308" rpy="0 0 0"/>

File: pick_robot_description/urdf/pick_robot.urdf.xacro (robot description, xacro)
@@ -168,8 +168,22 @@
     <origin xyz="0.0 0.0 0.01" rpy="0.0 0.0 ${pi}"/>
   </joint>
+  <!-- bracket/beugel -->
+  <xacro:include filename="beugel/urdf/Beugel.urdf.xacro" />
+  <xacro:include filename="beugel/urdf/BeugelWithArrow.urdf.xacro" />
+<!--
+  <xacro:beugel/>
+-->
+  <xacro:beugel_with_arrow/>
+  <!-- tool0 to beugel_base_position -->
+  <!-- cahnge these valuse to place the beugel on the right position -->
+  <joint name="beugel_base_position_to_tool0" type="fixed">
+    <parent link="tool0" />
+    <child link="beugel_base_link" />
+    <origin xyz="0.0 0.00 0.0" rpy="0 0 0"/>
+  </joint>
+  <!--
   <link name= "pick_tcp" />
-  <!-- bracket/beugel -->
-  <xacro:include filename="beugel/urdf/BeugelArrow.urdf.xacro" />
-  <xacro:beugel_arrow/>
+  -->
+<!--
   <joint name="pick_tcp_to_pick_tcp" type="fixed">
     <parent link="arrow_tcp" />
@@ -177,18 +191,8 @@
     <origin xyz="0.0 0.0 0.0" rpy="0.0 0.0 0.0"/>
   </joint>
-  <!--
-  <xacro:include filename="beugel/urdf/Beugel.urdf.xacro" />
-  <xacro:beugel/>
-  -->
-  <!-- tool0 to beugel_base_position -->
-  <!-- cahnge these valuse to place the beugel on the right position -->
-  <joint name="beugel_base_position_to_tool0" type="fixed">
-    <parent link="tool0" />
-    <child link="beugel_link" />
-    <origin xyz="0.0 0.00 0.0" rpy="0 0 0"/>
-  </joint>
+-->
     <xacro:arg name="camera_name"   default="oak" />
     <xacro:arg name="camera_model"  default="OAK-D" />
-    <xacro:arg name="base_frame"    default="beugel_camera" />
+    <xacro:arg name="base_frame"    default="beugel_camerax" />
     <xacro:arg name="parent_frame"  default="beugel_camera" />
     <xacro:arg name="cam_pos_x"     default="0.0" />
@@ -202,10 +206,8 @@
     <xacro:arg name="b"             default="0.0" />
     <xacro:arg name="a"             default="1.0" />
-<!--
     <xacro:include filename="$(find depthai_descriptions)/urdf/include/depthai_macro.urdf.xacro"/>
--->
     <xacro:include filename="depthai_macro.urdf.xacro"/>
     <xacro:depthai_camera camera_name = "$(arg camera_name)"
-parent = "$(arg parent_frame)"
+                          parent = "$(arg parent_frame)"
                           camera_model = "$(arg camera_model)"
                           base_frame = "$(arg base_frame)"
