Commit message: 20240412

File: pick_moveit_config/config/pick_robot.urdf.xacro (robot description, xacro)
@@ -1,7 +1,5 @@
 <?xml version="1.0"?>
 <robot xmlns:xacro="http://www.ros.org/wiki/xacro" name="pick_robot">
-    <!--
     <xacro:arg name="initial_positions_file" default="initial_positions.yaml" />
-    -->
     <!-- Import pick_robot urdf file -->
     <xacro:include filename="$(find pick_robot_description)/urdf/pick_robot.urdf.xacro" />

File: pick_robot_description/urdf/pick_robot.urdf.xacro (robot description, xacro)
@@ -127,4 +127,9 @@
       <xacro:box_inertia m="10" x="1.1" y="0.7" z="0.03"/>
     </inertial>
+    <collision>
+      <geometry>
+        <box size="0.7 1.1 0.03" />
+      </geometry>
+    </collision>
   </link>
   <joint name="baseplate_joint" type="fixed">
@@ -145,4 +150,9 @@
       <xacro:box_inertia m="1" x="0.3" y="0.3" z="0.012"/>
     </inertial>
+    <collision>
+      <geometry>
+        <box size="0.3 0.3 0.012" />
+      </geometry>
+    </collision>
   </link>
   <joint name="mountingplate_joint" type="fixed">
